File: lagom-main/PCB/_autosave-lagom.kicad_sch (KiCad schematic)
At the start: 171 parts, among them J1 Conn_01x04, J2 Conn_01x03, SW83 RotaryEncoder_Switch, SW84 RotaryEncoder_Switch, U2 74HC138, U3 74HC138, U5 Pico

Commit message: finalizing
Connections:
- net RotB: no longer D63.2 (A), D75.2 (A)
- new net: D63.2 (A), D75.2 (A)
Changed lines of the file:
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@@
-	)
-	(junction
-		(at 390.9296 108.9692)
-		(diameter 0)
-		(color 0 0 0 0)
 	)
 	(junction
@@
 	)
 	(junction
-		(at 375.666 114.8281)
-		(diameter 0)
-		(color 0 0 0 0)
-	)
-	(junction
 		(at 52.959 56.896)
 		(diameter 0)
@@
 	(wire
 		(pts
-			(xy 375.666 114.8281) (xy 390.9296 114.8281)
-		)
-		(stroke
-			(width 0)
-			(type default)
-		)
-	)
-	(wire
-		(pts
 			(xy 131.699 40.132) (xy 131.699 50.546)
 		)
@@
 		)
 		(stroke
-			(width 0)
-			(type default)
-		)
-	)
-	(wire
-		(pts
-			(xy 390.9296 108.9692) (xy 390.9296 114.8281)
-		)
-		(stroke
