File: lagom-main/PCB/lagom.kicad_pcb (KiCad board)
At the start: 2 copper layers, 426.6 x 122.7 mm, 179 parts, among them J1 Conn_01x04, J2 Conn_01x03, SW83 RotaryEncoder_Switch, SW84 RotaryEncoder_Switch, U1 ProMicro, U2 74HC138, U3 74HC138

Commit message: Changed PCB To Use a RPI Pico and Fixed Wiring Routes
Parts:
- removed the REF** at (392.4, 95.7)
- removed U1: ProMicro, Keebio-Parts:ArduinoProMicro-ZigZag
- added LCD1: LCD2.2", display:LCD2.2in, F.Cu at (390.5, 95.2)
- added U5: Pico, MCU_RaspberryPi_and_Boards:RPi_Pico_SMD_TH, F.Cu at (41.6, 48.2)
- SW_TAB1: footprint Button_Switch_Keyboard:SW_Cherry_MX_1.50u_PCB -> Button_Switch_Keyboard:SW_Cherry_MX_1.50u_Plate
- moved J1 54.3 mm to (369.4, 47.1)
Routing:
- net D/C(LCD): track 0.00 -> 661.1 mm, vias 0 -> 1
- net RST(LCD): track 0.00 -> 604.6 mm
- net CS(LCD): track 0.00 -> 597.7 mm
- net MOSI(LCD): track 0.00 -> 588.4 mm
- net SCK(LCD): track 0.00 -> 575.1 mm
- net GND: track 35.1 -> 515.6 mm
- net VCC: track 428.7 -> 681.3 mm, vias 1 -> 2
- net Net-(D16-K): track 65.5 -> 221.1 mm
- net Net-(D31-K): track 90.8 -> 210.7 mm
- net col14: track 318.3 -> 432.8 mm
- net Net-(D63-K): track 135.8 -> 233.7 mm
- net encA: track 263.2 -> 358.9 mm
- net SCL: track 253.5 -> 346.4 mm, vias 0 -> 1
- net RotB: track 321.6 -> 414.4 mm
- net encB: track 256.8 -> 349.3 mm
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Other:
- board size 426.6 x 122.7 mm -> 464.9 x 127.1 mm

Commit message: finalizing
Parts:
- added D75: D_Small, Diode_THT:D_DO-34_SOD68_P7.62mm_Horizontal, F.Cu at (293.7, 55.3)
- added RV1: R_Potentiometer, Potentiometer_THT:Potentiometer_Bourns_PTA6043_Single_Slide, F.Cu at (30.2, 76.9)
- added SW_DELETE1: KEYSW, Button_Switch_Keyboard:SW_Cherry_MX_1.00u_PCB, F.Cu at (448.8, 48.1)
- moved SW84 6.31 mm to (409.6, 50.1)
- moved SW_ENC2 6.31 mm to (412.2, 45.0)
Connections:
- D63 pad 2: row3 -> RotB
- U5 pad 29: unconnected-(U5-GPIO22-Pad29) -> Analogue
Routing:
- net Net-(D75-K): track 0.00 -> 160.5 mm, vias 0 -> 3
- net GND: track 515.6 -> 622.9 mm, vias 0 -> 1
- net Analogue: track 0.00 -> 86.5 mm
- net VCC: track 681.3 -> 727.7 mm
- net RotB: track 414.4 -> 457.8 mm, vias 0 -> 1
- net RotC: track 128.6 -> 136.5 mm
- net encD: track 367.1 -> 373.8 mm
- net encC: track 374.9 -> 381.2 mm
- net D/C(LCD): track 661.1 -> 658.6 mm
- net col12: track 363.6 -> 364.9 mm
- net RotA: track 111.0 -> 110.2 mm
Other:
- board size 464.9 x 127.1 mm -> 453.3 x 127.1 mm
- board text removed: "lagom v1"
